File: VideoJoystick/Schematic/FFJoystick/FFJoystick.kicad_sch (KiCad schematic)
At the start: 8 parts, among them J1 Raspberry_Pi_2_3, J2 Joystick Out, U1 LTC1661CN8-PBF, U2 RCD-24

Commit message: Updates to the schematic
Connections:
- net at J4.1 (Pin_1): no longer J1.32 (PWM0/GPIO12)
- net at R1.2, U2.3 (PWM/ON/OFF): now also J1.12 (GPIO18/PWM0); no longer J3.1 (Pin_1)
Changed lines of the file:
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@@
 		)
 		(stroke
-			(width 0)
-			(type default)
+			(width 0.381)
+			(type default)
+			(color 255 31 18 1)
 		)
 	)
@@
 	(wire
 		(pts
+			(xy 96.52 107.95) (xy 20.32 107.95)
+		)
+		(stroke
+			(width 0.254)
+			(type default)
+			(color 0 132 0 1)
+		)
+	)
+	(wire
+		(pts
+			(xy 20.32 107.95) (xy 20.32 46.99)
+		)
+		(stroke
+			(width 0.254)
+			(type default)
+			(color 0 132 0 1)
+		)
+	)
+	(wire
+		(pts
 			(xy 161.29 104.14) (xy 161.29 107.95)
 		)
@@
 	(wire
 		(pts
-			(xy 113.03 45.72) (xy 113.03 91.44)
-		)
-		(stroke
-			(width 0)
-			(type default)
-		)
-	)
-	(wire
-		(pts
 			(xy 86.36 67.31) (xy 71.12 67.31)
 		)
@@
 	(wire
 		(pts
-			(xy 107.95 45.72) (xy 113.03 45.72)
-		)
-		(stroke
-			(width 0)
-			(type default)
-		)
-	)
-	(wire
-		(pts
 			(xy 107.95 53.34) (xy 119.38 53.34)
 		)
@@
 	(wire
 		(pts
-			(xy 97.79 45.72) (xy 78.74 45.72)
-		)
-		(stroke
-			(width 0)
-			(type default)
-		)
-	)
-	(wire
-		(pts
 			(xy 208.28 46.99) (xy 229.87 46.99)
 		)
@@
 	(wire
 		(pts
-			(xy 78.74 45.72) (xy 78.74 74.93)
-		)
-		(stroke
-			(width 0)
-			(type default)
-		)
-	)
-	(wire
-		(pts
 			(xy 86.36 53.34) (xy 86.36 67.31)
 		)
@@
 	(wire
 		(pts
+			(xy 20.32 46.99) (xy 30.48 46.99)
+		)
+		(stroke
+			(width 0.254)
+			(type default)
+			(color 0 132 0 1)
+		)
+	)
+	(wire
+		(pts
 			(xy 93.98 48.26) (xy 93.98 62.23)
 		)
@@
 	(wire
 		(pts
-			(xy 113.03 91.44) (xy 127 91.44)
-		)
-		(stroke
-			(width 0)
-			(type default)
-		)
-	)
-	(wire
-		(pts
 			(xy 127 91.44) (xy 148.59 91.44)
 		)
@@
 	(wire
 		(pts
+			(xy 96.52 91.44) (xy 96.52 107.95)
+		)
+		(stroke
+			(width 0.254)
+			(type default)
+			(color 0 132 0 1)
+		)
+	)
+	(wire
+		(pts
 			(xy 81.28 50.8) (xy 81.28 69.85)
 		)
@@
 	(wire
 		(pts
-			(xy 78.74 74.93) (xy 71.12 74.93)
-		)
-		(stroke
-			(width 0)
-			(type default)
-		)
-	)
-	(wire
-		(pts
 			(xy 208.28 48.26) (xy 208.28 46.99)
 		)
@@
 		)
 		(stroke
-			(width 0)
-			(type default)
+			(width 0.381)
+			(type default)
+			(color 42 255 34 1)
 		)
 	)
@@
 		)
 	)
+	(wire
+		(pts
+			(xy 127 91.44) (xy 96.52 91.44)
+		)
+		(stroke
+			(width 0.254)
+			(type default)
+			(color 0 132 0 1)
+		)
+	)
